Commit message: [chore]: remove dummy elbow-end links LINK_ELBOW_END_L/R and joints J_FIXED_ELBOW_END_L/R

File: resource/robot/urdf/serial_pm_v2_identify.urdf (robot description, URDF)
Before this commit: robot pm_v2, 30 links, 29 joints
Links:
- removed link LINK_ELBOW_END_L
- removed link LINK_ELBOW_END_R
Joints:
- removed joint J_FIXED_ELBOW_END_L
- removed joint J_FIXED_ELBOW_END_R

Commit message: [feat]: add table environment for identification experiment

File: resource/robot/urdf/serial_pm_v2_identify.urdf (robot description, URDF)
Before this commit: robot pm_v2, 28 links, 27 joints
Links:
- added link table; collision box size=0.5 0.25 0.02; visual box size=0.5 0.25 0.02
- added link table_leg; collision box size=0.05 0.05 0.8; visual box size=0.05 0.05 0.8
Joints:
- added joint table: type fixed, parent lay_down, child table, origin xyz=-0.25 0 -0.11 rpy=0 0 0
- added joint table_leg: type fixed, parent lay_down, child table_leg, origin xyz=-0.025 0.1 -0.51 rpy=0 0 0

Commit message: [refactor]: reorder LINK_BASE definition and invert LAY_DOWN joint orientation

File: resource/robot/urdf/serial_pm_v2_identify.urdf (robot description, URDF)
Before this commit: robot pm_v2, 30 links, 29 joints
Joints:
- joint LAY_DOWN: child LINK_BASE -> lay_down; origin xyz=0 0 0 rpy=0 -1.57 0 -> xyz=0 0 0 rpy=0 1.57 0; parent lay_down -> LINK_BASE

Commit message: update table condition for leg

File: resource/robot/urdf/serial_pm_v2_identify.urdf (robot description, URDF)
Before this commit: robot pm_v2, 30 links, 29 joints
Links:
- added link table2; collision box size=0.8 0.25 0.02; visual box size=0.8 0.25 0.02
- link table: geometry collision box size=0.4 0.25 0.02; visual box size=0.4 0.25 0.02
Joints:
- added joint table2: type fixed, parent table, child table2, origin xyz=0.5 -0.1 0.0 rpy=0 0 -0.2
- joint table_leg: origin xyz=-0.025 0.1 -0.51 rpy=0 0 0 -> xyz=0.175 0.1 -0.4 rpy=0 0 0; parent lay_down -> table

Commit message: remove table leg

File: resource/robot/urdf/serial_pm_v2_identify.urdf (robot description, URDF)
Before this commit: robot pm_v2, 31 links, 30 joints
Links:
- removed link table_leg
Joints:
- removed joint table_leg
- joint table: origin xyz=-0.25 0 -0.11 rpy=0 0 0 -> xyz=-0.5 0 -0.11 rpy=0 0 0

Commit message: tune table size

File: resource/robot/urdf/serial_pm_v2_identify.urdf (robot description, URDF)
Before this commit: robot pm_v2, 30 links, 29 joints
Links:
- link table: geometry collision box size=0.8 0.25 0.02; visual box size=0.8 0.25 0.02
