Commit message: urdf used for simulation

File: resource/robot/urdf/serial_pm_v2_identify_true.urdf (robot description, URDF)
Before this commit: robot pm_v2, 28 links, 27 joints
Links:
- added link table; collision box size=0.8 0.25 0.02; visual box size=0.8 0.25 0.02
- added link table2; collision box size=0.8 0.25 0.02; visual box size=0.8 0.25 0.02
- link LINK_ANKLE_PITCH_L: mass 0.11534469 -> 0.11723776
- link LINK_ANKLE_PITCH_R: mass 0.11534469 -> 0.11705294
- link LINK_ANKLE_ROLL_L: mass 0.71786765 -> 0.73383772
- link LINK_ANKLE_ROLL_R: mass 0.71559163 -> 0.73297972
- link LINK_BASE: mass 4.08640035 -> 4.24027480
- link LINK_ELBOW_PITCH_L: mass 1.38061447 -> 1.44380190
- link LINK_ELBOW_PITCH_R: mass 1.38162913 -> 1.44600278
- link LINK_ELBOW_YAW_L: mass 0.46651916 -> 0.47172440
- link LINK_ELBOW_YAW_R: mass 0.46648073 -> 0.47211248
- link LINK_HEAD_YAW: mass 0.84510036 -> 0.87771797
- link LINK_HIP_PITCH_L: mass 1.68628239 -> 1.70994987
- link LINK_HIP_PITCH_R: mass 1.68024369 -> 1.69700932
- link LINK_HIP_ROLL_L: mass 0.63274283 -> 0.64685182
- link LINK_HIP_ROLL_R: mass 0.63673573 -> 0.64940150
- link LINK_HIP_YAW_L: mass 1.85800304 -> 1.93916783
- link LINK_HIP_YAW_R: mass 1.83146024 -> 1.91763466
- link LINK_KNEE_PITCH_L: mass 4.29474062 -> 4.47135738
- link LINK_KNEE_PITCH_R: mass 4.29186385 -> 4.46387469
- link LINK_SHOULDER_PITCH_L: mass 0.93215458 -> 0.94819020
- link LINK_SHOULDER_PITCH_R: mass 0.92914080 -> 0.94219549
- link LINK_SHOULDER_ROLL_L: mass 0.51081280 -> 0.52881636
- link LINK_SHOULDER_ROLL_R: mass 0.50967809 -> 0.52662000
- link LINK_SHOULDER_YAW_L: mass 0.90913792 -> 0.93921031
- link LINK_SHOULDER_YAW_R: mass 0.90851688 -> 0.93433519
- link LINK_TORSO_YAW: mass 9.01442210 -> 9.33297151
Joints:
- added joint table: type fixed, parent lay_down, child table, origin xyz=-0.5 0 -0.11 rpy=0 0 0
- added joint table2: type fixed, parent table, child table2, origin xyz=0.5 -0.1 0.0 rpy=0 0 -0.2
- joint LAY_DOWN: child LINK_BASE -> lay_down; origin xyz=0 0 0 rpy=0 -1.57 0 -> xyz=0 0 0 rpy=0 1.57 0; parent lay_down -> LINK_BASE
