Commit message: Adapt mesh path to new package structure

File: resource/robot/urdf/serial_pm_v2_command.urdf (robot description, URDF)
Before this commit: robot pm_v2, 29 links, 28 joints
Links:
- link command/LINK_ANKLE_PITCH_L: geometry collision mesh filename=package://identification/resource/robot/meshes/LINK_ANKLE_P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; visual mesh filename=package://identification/resource/robot/meshes/LINK_ANKLE_P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
- link command/LINK_ANKLE_PITCH_R: geometry collision mesh filename=package://identification/resource/robot/meshes/LINK_ANKLE_P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; visual mesh filename=package://identification/resource/robot/meshes/LINK_ANKLE_P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
- link command/LINK_ANKLE_ROLL_L: geometry collision mesh filename=package://identification/resource/robot/meshes/LINK_ANKLE_R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; visual mesh filename=package://identification/resource/robot/meshes/LINK_ANKLE_R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
- link command/LINK_ANKLE_ROLL_R: geometry collision mesh filename=package://identification/resource/robot/meshes/LINK_ANKLE_R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; visual mesh filename=package://identification/resource/robot/meshes/LINK_ANKLE_R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
- link command/LINK_BASE: geometry collision mesh filename=package://identification/resource/robot/meshes/LINK_BASE.STL; visual mesh filename=package://identification/resource/robot/meshes/LINK_BASE.STL
- link command/LINK_ELBOW_PITCH_L: geometry collision mesh filename=package://identification/resource/robot/meshes/LINK_ELBOW_P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; visual mesh filename=package://identification/resource/robot/meshes/LINK_ELBOW_P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
- link command/LINK_ELBOW_PITCH_R: geometry collision mesh filename=package://identification/resource/robot/meshes/LINK_ELBOW_P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; visual mesh filename=package://identification/resource/robot/meshes/LINK_ELBOW_P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
- link command/LINK_ELBOW_YAW_L: geometry collision mesh filename=package://identification/resource/robot/meshes/LINK_ELBOW_Y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; visual mesh filename=package://identification/resource/robot/meshes/LINK_ELBOW_Y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
- link command/LINK_ELBOW_YAW_R: geometry collision mesh filename=package://identification/resource/robot/meshes/LINK_ELBOW_Y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; visual mesh filename=package://identification/resource/robot/meshes/LINK_ELBOW_Y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
- link command/LINK_HEAD_YAW: geometry collision mesh filename=package://identification/resource/robot/meshes/LINK_HEAD_YA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; visual mesh filename=package://identification/resource/robot/meshes/LINK_HEAD_YA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
- link command/LINK_HIP_PITCH_L: geometry collision mesh filename=package://identification/resource/robot/meshes/LINK_HIP_PIT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; visual mesh filename=package://identification/resource/robot/meshes/LINK_HIP_PIT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
- link command/LINK_HIP_PITCH_R: geometry collision mesh filename=package://identification/resource/robot/meshes/LINK_HIP_PIT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; visual mesh filename=package://identification/resource/robot/meshes/LINK_HIP_PIT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
- link command/LINK_HIP_ROLL_L: geometry collision mesh filename=package://identification/resource/robot/meshes/LINK_HIP_ROL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; visual mesh filename=package://identification/resource/robot/meshes/LINK_HIP_ROL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
- link command/LINK_HIP_ROLL_R: geometry collision mesh filename=package://identification/resource/robot/meshes/LINK_HIP_ROL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; visual mesh filename=package://identification/resource/robot/meshes/LINK_HIP_ROL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
- link command/LINK_HIP_YAW_L: geometry collision mesh filename=package://identification/resource/robot/meshes/LINK_HIP_YAW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; visual mesh filename=package://identification/resource/robot/meshes/LINK_HIP_YAW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
- link command/LINK_HIP_YAW_R: geometry collision mesh filename=package://identification/resource/robot/meshes/LINK_HIP_YAW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; visual mesh filename=package://identification/resource/robot/meshes/LINK_HIP_YAW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
- link command/LINK_KNEE_PITCH_L: geometry collision mesh filename=package://identification/resource/robot/meshes/LINK_KNEE_PI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; visual mesh filename=package://identification/resource/robot/meshes/LINK_KNEE_PI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
- link command/LINK_KNEE_PITCH_R: geometry collision mesh filename=package://identification/resource/robot/meshes/LINK_KNEE_PI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; visual mesh filename=package://identification/resource/robot/meshes/LINK_KNEE_PI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
- link command/LINK_SHOULDER_PITCH_L: geometry collision mesh filename=package://identification/resource/robot/meshes/LINK_SHOULDE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; visual mesh filename=package://identification/resource/robot/meshes/LINK_SHOULDE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
- link command/LINK_SHOULDER_PITCH_R: geometry collision mesh filename=package://identification/resource/robot/meshes/LINK_SHOULDE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; visual mesh filename=package://identification/resource/robot/meshes/LINK_SHOULDE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
- link command/LINK_SHOULDER_ROLL_L: geometry collision mesh filename=package://identification/resource/robot/meshes/LINK_SHOULDE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; visual mesh filename=package://identification/resource/robot/meshes/LINK_SHOULDE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
- link command/LINK_SHOULDER_ROLL_R: geometry collision mesh filename=package://identification/resource/robot/meshes/LINK_SHOULDE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; visual mesh filename=package://identification/resource/robot/meshes/LINK_SHOULDE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
- link command/LINK_SHOULDER_YAW_L: geometry collision mesh filename=package://identification/resource/robot/meshes/LINK_SHOULDE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; visual mesh filename=package://identification/resource/robot/meshes/LINK_SHOULDE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
- link command/LINK_SHOULDER_YAW_R: geometry collision mesh filename=package://identification/resource/robot/meshes/LINK_SHOULDE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; visual mesh filename=package://identification/resource/robot/meshes/LINK_SHOULDE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
- link command/LINK_TORSO_YAW: geometry collision mesh filename=package://identification/resource/robot/meshes/LINK_TORSO_Y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; visual mesh filename=package://identification/resource/robot/meshes/LINK_TORSO_Y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
