Commit message: model used

File: resource/robot/urdf/serial_pm_v2_identify_flat.urdf (robot description, URDF)
Before this commit: robot pm_v2, 30 links, 29 joints
Links:
- link LINK_ANKLE_PITCH_L: mass 0.14351955 -> 0.11534469
- link LINK_ANKLE_PITCH_R: mass 0.13875665 -> 0.11534469
- link LINK_ANKLE_ROLL_L: mass 0.90424401 -> 0.71786765
- link LINK_ANKLE_ROLL_R: mass 0.88433216 -> 0.71559163
- link LINK_BASE: mass 5.06943990 -> 4.08640035
- link LINK_ELBOW_PITCH_L: mass 1.65291080 -> 1.70200160
- link LINK_ELBOW_PITCH_R: mass 1.73731444 -> 1.38162913
- link LINK_ELBOW_YAW_L: mass 0.57211986 -> 0.66089632
- link LINK_ELBOW_YAW_R: mass 0.59712586 -> 0.46648073
- link LINK_HEAD_YAW: mass 1.08639099 -> 0.84510036
- link LINK_HIP_PITCH_L: mass 2.04513409 -> 1.68628239
- link LINK_HIP_PITCH_R: mass 2.06525049 -> 1.68024369
- link LINK_HIP_ROLL_L: mass 0.80625250 -> 0.63274283
- link LINK_HIP_ROLL_R: mass 0.80843716 -> 0.63673573
- link LINK_HIP_YAW_L: mass 2.29780105 -> 1.85800304
- link LINK_HIP_YAW_R: mass 2.15341849 -> 1.83146024
- link LINK_KNEE_PITCH_L: mass 5.17662951 -> 4.29474062
- link LINK_KNEE_PITCH_R: mass 5.05821641 -> 4.29186385
- link LINK_SHOULDER_PITCH_L: mass 1.14093594 -> 0.93215458
- link LINK_SHOULDER_PITCH_R: mass 1.12703857 -> 0.92914080
- link LINK_SHOULDER_ROLL_L: mass 0.63147420 -> 0.48324268
- link LINK_SHOULDER_ROLL_R: mass 0.62310500 -> 0.50967809
- link LINK_SHOULDER_YAW_L: mass 1.09934346 -> 1.03575756
- link LINK_SHOULDER_YAW_R: mass 1.14691096 -> 0.90851688
- link LINK_TORSO_YAW: mass 10.76940175 -> 9.01442210

File: resource/robot/urdf/serial_pm_v2_identify_result_arm.urdf (robot description, URDF)
Before this commit: robot pm_v2, 30 links, 29 joints
Links:
- link LINK_ANKLE_PITCH_L: mass 0.14351955 -> 0.11534469
- link LINK_ANKLE_PITCH_R: mass 0.13875665 -> 0.11534469
- link LINK_ANKLE_ROLL_L: mass 0.90424401 -> 0.71786765
- link LINK_ANKLE_ROLL_R: mass 0.88433216 -> 0.71559163
- link LINK_BASE: mass 5.06943990 -> 4.08640035
- link LINK_ELBOW_PITCH_L: mass 1.65291080 -> 1.29613452
- link LINK_ELBOW_PITCH_R: mass 1.73731444 -> 1.38162913
- link LINK_ELBOW_YAW_L: mass 0.57211986 -> 0.35127656
- link LINK_ELBOW_YAW_R: mass 0.59712586 -> 0.46648073
- link LINK_HEAD_YAW: mass 1.08639099 -> 0.84510036
- link LINK_HIP_PITCH_L: mass 2.04513409 -> 1.68628239
- link LINK_HIP_PITCH_R: mass 2.06525049 -> 1.68024369
- link LINK_HIP_ROLL_L: mass 0.80625250 -> 0.63274283
- link LINK_HIP_ROLL_R: mass 0.80843716 -> 0.63673573
- link LINK_HIP_YAW_L: mass 2.29780105 -> 1.85800304
- link LINK_HIP_YAW_R: mass 2.15341849 -> 1.83146024
- link LINK_KNEE_PITCH_L: mass 5.17662951 -> 4.29474062
- link LINK_KNEE_PITCH_R: mass 5.05821641 -> 4.29186385
- link LINK_SHOULDER_PITCH_L: mass 1.14093594 -> 0.93215457
- link LINK_SHOULDER_PITCH_R: mass 1.12703857 -> 0.92914080
- link LINK_SHOULDER_ROLL_L: mass 0.63147420 -> 0.55133949
- link LINK_SHOULDER_ROLL_R: mass 0.62310500 -> 0.50967809
- link LINK_SHOULDER_YAW_L: mass 1.09934346 -> 0.93222052
- link LINK_SHOULDER_YAW_R: mass 1.14691096 -> 0.90851688
- link LINK_TORSO_YAW: mass 10.76940175 -> 9.01442210
