Commit message: urdf identified results

File: resource/robot/urdf/serial_pm_v2_identify_sim_arm.urdf (robot description, URDF)
Before this commit: robot pm_v2, 30 links, 29 joints
Links:
- link LINK_ELBOW_PITCH_L: mass 1.29613452 -> 1.70182598
- link LINK_ELBOW_YAW_L: mass 0.35127656 -> 0.66267869
- link LINK_SHOULDER_PITCH_L: mass 0.93215457 -> 0.93215458
- link LINK_SHOULDER_ROLL_L: mass 0.55133949 -> 0.48180635
- link LINK_SHOULDER_YAW_L: mass 0.93222052 -> 1.03274932
