Commit message: sim identified result leg

File: resource/robot/urdf/serial_pm_v2_identify_sim_leg.urdf (robot description, URDF)
Before this commit: robot pm_v2, 30 links, 29 joints
Links:
- link LINK_ANKLE_PITCH_L: mass 0.11598679 -> 0.11034853
- link LINK_ANKLE_ROLL_L: mass 0.74198853 -> 0.76462791
- link LINK_HIP_ROLL_L: mass 0.69765009 -> 0.67890190
- link LINK_HIP_YAW_L: mass 2.24915685 -> 2.19717081
- link LINK_KNEE_PITCH_L: mass 5.46857805 -> 5.46181275

Commit message: update identified URDF results

File: resource/robot/urdf/serial_pm_v2_identify_sim_leg.urdf (robot description, URDF)
Before this commit: robot pm_v2, 30 links, 29 joints
Links:
- link LINK_ANKLE_PITCH_L: mass 0.11034853 -> 0.11819858
- link LINK_ANKLE_ROLL_L: mass 0.76462791 -> 0.79751548
- link LINK_HIP_PITCH_L: mass 1.68628239 -> 1.68628238
- link LINK_HIP_ROLL_L: mass 0.67890190 -> 0.64648841
- link LINK_HIP_YAW_L: mass 2.19717081 -> 2.08230357
- link LINK_KNEE_PITCH_L: mass 5.46181275 -> 5.44465909
